Commit message: First working igus rebel description WS :))

File: ros2_dev_ws/src/igus_rebel_description/urdf/igus_rebel.urdf (robot description, URDF)
Before this commit: robot igus_rebel, 9 links, 8 joints
Links:
- link base_link: geometry collision mesh filename=package://igus_rebel_description/meshes/Robolink_RebeL_000.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; visual mesh filename=package://igus_rebel_description/meshes/Robolink_RebeL_000.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
- link link_1: geometry collision mesh filename=package://igus_rebel_description/meshes/Robolink_RebeL_001.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; visual mesh filename=package://igus_rebel_description/meshes/Robolink_RebeL_001.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
- link link_2: geometry collision mesh filename=package://igus_rebel_description/meshes/Robolink_RebeL_002_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; visual mesh filename=package://igus_rebel_description/meshes/Robolink_RebeL_002_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
- link link_3: geometry collision mesh filename=package://igus_rebel_description/meshes/Robolink_RebeL_002_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; visual mesh filename=package://igus_rebel_description/meshes/Robolink_RebeL_002_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
- link link_4: geometry collision mesh filename=package://igus_rebel_description/meshes/Robolink_RebeL_002_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; visual mesh filename=package://igus_rebel_description/meshes/Robolink_RebeL_002_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
- link link_5: geometry collision mesh filename=package://igus_rebel_description/meshes/Robolink_RebeL_003.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; visual mesh filename=package://igus_rebel_description/meshes/Robolink_RebeL_003.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
- link link_6: geometry collision mesh filename=package://igus_rebel_description/meshes/Robolink_RebeL_004.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; visual mesh filename=package://igus_rebel_description/meshes/Robolink_RebeL_004.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
- link link_7: geometry collision mesh filename=package://igus_rebel_description/meshes/Robolink_RebeL_005.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; visual mesh filename=package://igus_rebel_description/meshes/Robolink_RebeL_005.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
- link link_8: geometry collision mesh filename=package://igus_rebel_description/meshes/Robolink_RebeL_006.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; visual mesh filename=package://igus_rebel_description/meshes/Robolink_RebeL_006.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

File: ros2_dev_ws/src/rebel_test/urdf/rebel.urdf (robot description, URDF)
Before this commit: robot igus_rebel, 2 links, 1 joints
Links:
- link base_link: geometry visual mesh filename=package://rebel_test/meshes/test.dae
- link world: geometry visual mesh filename=package://rebel_test/meshes/test.stl
